File: V1/UKHASnet-avr-sensor.brd (EAGLE design)
At the start: 49.5 x 49.2 mm, 23 parts, among them J1 AVR_SPI_PRG_62X3_LOCK, U1 MCP1700-3302E/TO, U2 ATMEGA328P-PU, Y1 RESONATORPTH

Commit message: More little tweaks, send it off to Mitch!
Parts:
- added JP12, JP13, JP14: M01PTH, SparkFun-Connectors:1X01
Connections:
- new net N$12: JP14.1, U2.2
- new net N$13: JP13.1, U2.3
- net GND: now also JP12.1
Routing:
- net N$13: track 0.00 -> 3.81 mm
- net N$12: track 0.00 -> 3.81 mm
Changed lines of the file:
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@@
 <element name="R4" library="SparkFun" package="AXIAL-0.4" value="" x="10.16" y="5.08" rot="R180"/>
 <element name="Y1" library="SparkFun" package="RESONATOR-PTH" value="RESONATORPTH" x="2.54" y="19.05" rot="R270"/>
+<element name="JP12" library="SparkFun-Connectors" package="1X01" value="M01PTH" x="2.54" y="33.02" smashed="yes"/>
+<element name="JP13" library="SparkFun-Connectors" package="1X01" value="M01PTH" x="2.54" y="35.56" smashed="yes"/>
+<element name="JP14" library="SparkFun-Connectors" package="1X01" value="M01PTH" x="2.54" y="38.1" smashed="yes"/>
 </elements>
 <signals>
@@
 <via x="8.89" y="44.45" extent="1-16" drill="0.6"/>
 <via x="1.27" y="43.18" extent="1-16" drill="0.6"/>
-<via x="1.27" y="39.37" extent="1-16" drill="0.6"/>
-<via x="1.27" y="35.56" extent="1-16" drill="0.6"/>
-<via x="1.27" y="31.75" extent="1-16" drill="0.6"/>
+<via x="2.54" y="40.64" extent="1-16" drill="0.6"/>
+<via x="3.81" y="43.18" extent="1-16" drill="0.6"/>
+<via x="43.18" y="45.72" extent="1-16" drill="0.6"/>
 <via x="1.27" y="23.495" extent="1-16" drill="0.6"/>
 <via x="5.08" y="19.05" extent="1-16" drill="0.6"/>
@@
 <via x="24.13" y="1.27" extent="1-16" drill="0.6"/>
 <contactref element="Y1" pad="2"/>
+<contactref element="JP12" pad="1"/>
 </signal>
 <signal name="VIN">
@@
 <wire x1="10.16" y1="29.21" x2="6.35" y2="33.02" width="0.4064" layer="16"/>
 </signal>
+<signal name="N$12">
+<contactref element="JP14" pad="1"/>
+<contactref element="U2" pad="2"/>
+<wire x1="6.35" y1="38.1" x2="2.54" y2="38.1" width="0.4064" layer="1"/>
+</signal>
+<signal name="N$13">
+<contactref element="U2" pad="3"/>
+<contactref element="JP13" pad="1"/>
+<wire x1="6.35" y1="35.56" x2="2.54" y2="35.56" width="0.4064" layer="1"/>
+</signal>
 </signals>
