File: V2/UKHASnet-avr-sensor.sch (EAGLE design)
At the start: 33 parts, among them J1 AVR_SPI_PRG_62X3_LOCK, U1 MCP1700-3302E/TO, U2 ATMEGA328P-PU, X1 SMA-142-0711-881/886, Y1 RESONATORPTH

Commit message: Drive sensor vcc from AVR PB0.
Parts:
- added C7: 0.1uF, capacitor-wima:C2.5/2
Connections:
- new net SENSE_VCC: C7.1, R4.2, U$2.VCC, U2.PB0
- net GND: now also C7.2
- net VCC: no longer R4.2, U$2.VCC
Changed lines of the file:
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@@
 <part name="JP15" library="SparkFun-Connectors" deviceset="M01" device="PTH"/>
 <part name="PAD1" library="wirepad" deviceset="WIREPAD" device="1,6/0,9"/>
+<part name="C7" library="capacitor-wima" deviceset="C" device="2.5/2" value="0.1uF"/>
 </parts>
 <sheets>
@@
 <instance part="JP15" gate="G$1" x="144.78" y="83.82" rot="R180"/>
 <instance part="PAD1" gate="G$1" x="-15.24" y="33.02"/>
+<instance part="C7" gate="G$1" x="15.24" y="50.8"/>
 </instances>
 <busses>
@@
 <wire x1="15.24" y1="101.6" x2="15.24" y2="104.14" width="0.1524" layer="91"/>
 <junction x="15.24" y="104.14"/>
-</segment>
-<segment>
-<pinref part="U$2" gate="G$1" pin="VCC"/>
-<wire x1="-7.62" y1="48.26" x2="-5.08" y2="48.26" width="0.1524" layer="91"/>
-<wire x1="-5.08" y1="48.26" x2="-5.08" y2="55.88" width="0.1524" layer="91"/>
-<wire x1="-5.08" y1="55.88" x2="0" y2="55.88" width="0.1524" layer="91"/>
-<pinref part="R4" gate="G$1" pin="2"/>
-<wire x1="10.16" y1="55.88" x2="0" y2="55.88" width="0.1524" layer="91"/>
-<junction x="0" y="55.88"/>
-<label x="5.08" y="55.88" size="1.778" layer="95"/>
 </segment>
 <segment>
@@
 <wire x1="-7.62" y1="43.18" x2="-2.54" y2="43.18" width="0.1524" layer="91"/>
 <label x="5.08" y="43.18" size="1.778" layer="95"/>
-<wire x1="-2.54" y1="43.18" x2="10.16" y2="43.18" width="0.1524" layer="91"/>
+<wire x1="-2.54" y1="43.18" x2="15.24" y2="43.18" width="0.1524" layer="91"/>
 <wire x1="-12.7" y1="33.02" x2="-2.54" y2="33.02" width="0.1524" layer="91"/>
 <wire x1="-2.54" y1="33.02" x2="-2.54" y2="43.18" width="0.1524" layer="91"/>
 <junction x="-2.54" y="43.18"/>
 <pinref part="PAD1" gate="G$1" pin="P"/>
+<pinref part="C7" gate="G$1" pin="2"/>
+<wire x1="15.24" y1="45.72" x2="15.24" y2="43.18" width="0.1524" layer="91"/>
 </segment>
 <segment>
@@
 </segment>
 </net>
+<net name="SENSE_VCC" class="0">
+<segment>
+<pinref part="U2" gate="A" pin="PB0"/>
+<wire x1="53.34" y1="58.42" x2="40.64" y2="58.42" width="0.1524" layer="91"/>
+<label x="43.18" y="58.42" size="1.778" layer="95"/>
+</segment>
+<segment>
+<pinref part="U$2" gate="G$1" pin="VCC"/>
+<wire x1="-7.62" y1="48.26" x2="-5.08" y2="48.26" width="0.1524" layer="91"/>
+<wire x1="-5.08" y1="48.26" x2="-5.08" y2="55.88" width="0.1524" layer="91"/>
+<wire x1="-5.08" y1="55.88" x2="0" y2="55.88" width="0.1524" layer="91"/>
+<pinref part="R4" gate="G$1" pin="2"/>
+<wire x1="15.24" y1="55.88" x2="0" y2="55.88" width="0.1524" layer="91"/>
+<junction x="0" y="55.88"/>
+<label x="-5.08" y="55.88" size="1.778" layer="95"/>
+<pinref part="C7" gate="G$1" pin="1"/>
+<wire x1="15.24" y1="53.34" x2="15.24" y2="55.88" width="0.1524" layer="91"/>
+</segment>
+</net>
