File: V3/UKHASnet-avr-sensor.brd (EAGLE design)
At the start: 49.5 x 49.2 mm, 26 parts, among them J1 AVR_SPI_PRG_62X3_LOCK, U1 MCP1700-3302E/TO, U2 ATMEGA328P-PU, X2 SMA-142-0711-821/826, Y1 RESONATORPTH

Commit message: Adjust V3 Silkscreen.
Parts:
- moved JP6 0.63 mm to (14.9, 1.59)
Other:
- board text added: "18B20/DHT22"
Changed lines of the file:
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@@
 <wire x1="2" y1="49.2" x2="0" y2="47.2" width="0" layer="20" curve="90"/>
 <text x="41.91" y="10.16" size="1.778" layer="51" distance="96" rot="R90">Phil M0DNY</text>
-<text x="24.765" y="12.7" size="1.778" layer="51" rot="R90">https://ukhas.net/</text>
+<text x="24.765" y="13.97" size="1.778" layer="51" rot="R90">https://ukhas.net/</text>
 <text x="41.91" y="1.27" size="1.9304" layer="51">+</text>
 <text x="36.83" y="10.16" size="1.778" layer="51" rot="R90">Sensor V3</text>
@@
 <text x="3.175" y="30.7975" size="1.27" layer="51">+</text>
 <text x="43.18" y="3.81" size="1.016" layer="51">max 6V</text>
+<text x="13.97" y="3.175" size="1.016" layer="51">18B20/DHT22</text>
 </plain>
 <attributes>
@@
 <attribute name="SUPPLIER" value="PANASONIC " x="25.4" y="6.35" size="1.778" layer="27" rot="R90" display="off"/>
 <attribute name="OC_FARNELL" value="1848468 " x="25.4" y="6.35" size="1.778" layer="27" rot="R90" display="off"/>
-<attribute name="VALUE" x="19.7358" y="4.9784" size="0.8128" layer="27" font="vector" ratio="15" rot="SR0"/>
+<attribute name="VALUE" x="20.0533" y="5.9309" size="0.8128" layer="27" font="vector" ratio="15" rot="SR0"/>
 </element>
 <element name="R4" library="SparkFun" package="AXIAL-0.4" value="4.7K" x="7.62" y="5.08" smashed="yes">
@@
 <attribute name="OC_FARNELL" value="1019328" x="24.765" y="49.2125" size="1.778" layer="27" rot="R270" display="off"/>
 </element>
-<element name="JP6" library="SparkFun-Connectors" package="1X04" value="" x="14.2875" y="1.5875" smashed="yes">
-<attribute name="VALUE" x="13.0175" y="-1.5875" size="1.27" layer="27"/>
+<element name="JP6" library="SparkFun-Connectors" package="1X04" value="" x="14.9225" y="1.5875" smashed="yes">
+<attribute name="VALUE" x="13.6525" y="-1.5875" size="1.27" layer="27"/>
 </element>
 </elements>
@@
 <contactref element="R4" pad="P$1"/>
 <wire x1="9.525" y1="5.08" x2="2.54" y2="5.08" width="0.4064" layer="16"/>
-<wire x1="16.8275" y1="4.7625" x2="13.97" y2="7.62" width="0.4064" layer="1"/>
+<wire x1="17.4625" y1="4.1275" x2="13.97" y2="7.62" width="0.4064" layer="1"/>
 <contactref element="JP6" pad="2"/>
-<wire x1="16.8275" y1="1.5875" x2="16.8275" y2="4.7625" width="0.4064" layer="1"/>
+<wire x1="17.4625" y1="1.5875" x2="17.4625" y2="4.1275" width="0.4064" layer="1"/>
 </signal>
 <signal name="GND">
@@
 <via x="7.62" y="0.635" extent="1-16" drill="0.3"/>
 <via x="10.16" y="0.635" extent="1-16" drill="0.3"/>
-<via x="12.7" y="0.635" extent="1-16" drill="0.3"/>
-<via x="18.0975" y="3.175" extent="1-16" drill="0.3"/>
+<via x="12.3825" y="0.635" extent="1-16" drill="0.3"/>
+<via x="18.7325" y="3.175" extent="1-16" drill="0.3"/>
 <via x="4.445" y="6.35" extent="1-16" drill="0.3"/>
 <via x="9.2075" y="6.35" extent="1-16" drill="0.3"/>
-<via x="22.86" y="0.635" extent="1-16" drill="0.3"/>
-<via x="25.4" y="0.635" extent="1-16" drill="0.3"/>
-<via x="27.94" y="0.635" extent="1-16" drill="0.3"/>
-<via x="30.48" y="0.635" extent="1-16" drill="0.3"/>
-<via x="33.02" y="0.635" extent="1-16" drill="0.3"/>
-<via x="35.56" y="0.635" extent="1-16" drill="0.3"/>
-<via x="38.1" y="0.635" extent="1-16" drill="0.3"/>
+<via x="24.765" y="0.635" extent="1-16" drill="0.3"/>
+<via x="27.305" y="7.62" extent="1-16" drill="0.3"/>
+<via x="27.6225" y="0.635" extent="1-16" drill="0.3"/>
+<via x="31.115" y="0.635" extent="1-16" drill="0.3"/>
+<via x="34.6075" y="0.635" extent="1-16" drill="0.3"/>
+<via x="2.2225" y="40.005" extent="1-16" drill="0.3"/>
+<via x="37.7825" y="0.635" extent="1-16" drill="0.3"/>
 <via x="40.64" y="0.635" extent="1-16" drill="0.3"/>
 <via x="43.18" y="0.635" extent="1-16" drill="0.3"/>
@@
 <via x="48.895" y="10.16" extent="1-16" drill="0.3"/>
 <via x="37.465" y="3.81" extent="1-16" drill="0.3"/>
-<via x="35.56" y="3.175" extent="1-16" drill="0.3"/>
+<via x="34.6075" y="3.175" extent="1-16" drill="0.3"/>
 <via x="37.465" y="6.985" extent="1-16" drill="0.3"/>
 <via x="37.7825" y="13.97" extent="1-16" drill="0.3"/>
@@
 <via x="23.495" y="42.2275" extent="1-16" drill="0.3"/>
 <via x="7.62" y="3.175" extent="1-16" drill="0.3"/>
-<via x="12.7" y="3.175" extent="1-16" drill="0.3"/>
+<via x="12.3825" y="3.175" extent="1-16" drill="0.3"/>
 <via x="16.8275" y="7.3025" extent="1-16" drill="0.3"/>
 <via x="19.05" y="7.3025" extent="1-16" drill="0.3"/>
@@
 <via x="14.605" y="5.08" extent="1-16" drill="0.3"/>
 <via x="18.0975" y="5.3975" extent="1-16" drill="0.3"/>
-<via x="24.13" y="2.54" extent="1-16" drill="0.3"/>
-<via x="26.67" y="2.54" extent="1-16" drill="0.3"/>
+<via x="33.9725" y="12.7" extent="1-16" drill="0.3"/>
+<via x="27.6225" y="2.54" extent="1-16" drill="0.3"/>
 <via x="34.29" y="7.62" extent="1-16" drill="0.3"/>
 <via x="36.83" y="8.255" extent="1-16" drill="0.3"/>
@@
 <wire x1="12.7" y1="5.08" x2="8.89" y2="5.08" width="0.4064" layer="1"/>
 <wire x1="8.89" y1="5.08" x2="6.35" y2="7.62" width="0.4064" layer="1"/>
-<wire x1="12.7" y1="5.08" x2="14.2875" y2="3.4925" width="0.4064" layer="1"/>
+<wire x1="12.7" y1="5.08" x2="14.9225" y2="2.8575" width="0.4064" layer="1"/>
 <contactref element="JP6" pad="1"/>
-<wire x1="14.2875" y1="1.5875" x2="14.2875" y2="3.4925" width="0.4064" layer="1"/>
+<wire x1="14.9225" y1="1.5875" x2="14.9225" y2="2.8575" width="0.4064" layer="1"/>
 </signal>
 </signals>
