File: uV1/UKHASnet-avr-sensor.brd (EAGLE design)
At the start: 37.8 x 44.4 mm, 14 parts, among them J1 AVR_SPI_PRG_62X3_LOCK, U2 ATMEGA328P-AU

Commit message: Not much progress.
Parts:
- removed U$2: DS1820TO92, Ava:DS1820
- added JP4: (no value), SparkFun-Connectors:1X04
Connections:
- net GND: no longer U$2.GND
- net SENSE1: no longer U$2.DQ
- net SENSE_VCC: no longer U$2.VDD
Routing:
- net SCK: track 27.3 -> 29.1 mm
- net SENSE1: track 6.59 -> 5.02 mm
- net SENSE_VCC: track 7.04 -> 6.17 mm
Changed lines of the file:
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@@
 <elements>
 <element name="U$1" library="hopeRF2" package="RFM" value="RFM69HW" x="15.5575" y="2.2225" smashed="yes"/>
-<element name="U$2" library="Ava" package="DS1820" value="DS1820TO92" x="22.225" y="2.2225" smashed="yes"/>
 <element name="J1" library="SparkFun-Connectors" package="2X3_LOCK" value="AVR_SPI_PRG_62X3_LOCK" x="1.905" y="12.3825" smashed="yes" rot="R270"/>
 <element name="U2" library="Ava" package="QFP80P900X900X120-32N" value="ATMEGA328P-AU" x="25.0825" y="11.7475" smashed="yes" rot="MR0">
@@
 <element name="JP1" library="SparkFun-Connectors" package="1X01" value="M01PTH" x="31.115" y="0.9525" smashed="yes"/>
 <element name="JP3" library="SparkFun-Connectors" package="1X01" value="M01PTH" x="20.0025" y="0.9525" smashed="yes"/>
+<element name="JP4" library="SparkFun-Connectors" package="1X04" value="" x="27.6225" y="22.225"/>
 </elements>
 <signals>
@@
 <wire x1="1.651" y1="9.8425" x2="1.905" y2="9.8425" width="0.254" layer="16"/>
 <wire x1="1.905" y1="9.8425" x2="3.175" y2="8.5725" width="0.254" layer="16"/>
-<wire x1="3.175" y1="8.5725" x2="11.7475" y2="8.5725" width="0.254" layer="16"/>
-<wire x1="11.7475" y1="8.5725" x2="20.8407" y2="8.9535" width="0" layer="19" extent="16-16"/>
+<wire x1="3.175" y1="8.5725" x2="13.0175" y2="8.5725" width="0.254" layer="16"/>
+<wire x1="13.0175" y1="8.5725" x2="13.335" y2="8.255" width="0.254" layer="16"/>
+<wire x1="13.335" y1="8.255" x2="20.8407" y2="8.9535" width="0" layer="19" extent="16-16"/>
 </signal>
 <signal name="MISO">
@@
 <signal name="SENSE1">
 <contactref element="U2" pad="13"/>
-<contactref element="U$2" pad="DQ"/>
 <contactref element="R1" pad="2"/>
 <wire x1="24.6761" y1="7.5057" x2="24.75" y2="7.4318" width="0.254" layer="16" curve="-90"/>
 <wire x1="24.75" y1="7.4318" x2="24.75" y2="2.54" width="0.254" layer="16"/>
 <wire x1="24.75" y1="2.54" x2="24.765" y2="2.525" width="0.254" layer="16" curve="-90"/>
-<wire x1="24.765" y1="2.525" x2="24.765" y2="0.9525" width="0.254" layer="16"/>
 </signal>
 <signal name="GND">
-<polygon width="0.4064" layer="16">
-<vertex x="3.81" y="20.0025"/>
-<vertex x="39.0525" y="19.685"/>
+<polygon width="0.4064" layer="16" isolate="0.254">
+<vertex x="13.97" y="17.78"/>
+<vertex x="38.735" y="17.78"/>
 <vertex x="39.0525" y="6.0325"/>
 <vertex x="38.735" y="5.715"/>
 <vertex x="38.735" y="-0.9525"/>
 <vertex x="36.5125" y="-0.9525"/>
-<vertex x="3.4925" y="-1.5875"/>
+<vertex x="13.97" y="-2.2225"/>
 </polygon>
-<polygon width="0.4064" layer="1">
-<vertex x="3.81" y="20.0025"/>
-<vertex x="39.0525" y="19.3675"/>
+<polygon width="0.4064" layer="1" isolate="0.254">
+<vertex x="13.97" y="17.78"/>
+<vertex x="38.735" y="17.78"/>
 <vertex x="39.0525" y="-2.54"/>
-<vertex x="3.81" y="-0.9525"/>
+<vertex x="13.97" y="-1.5875"/>
 </polygon>
 <contactref element="J1" pad="6"/>
@@
 <contactref element="U$1" pad="GNDB"/>
 <contactref element="U2" pad="3"/>
-<contactref element="U$2" pad="GND"/>
 <contactref element="U2" pad="21"/>
 <contactref element="U2" pad="5"/>
 <wire x1="4.445" y1="7.3025" x2="13.0175" y2="7.3025" width="0.254" layer="16"/>
 <via x="14.9225" y="0.635" extent="1-16" drill="0.5" diameter="0.254"/>
-<via x="14.9225" y="18.7325" extent="1-16" drill="0.5" diameter="0.254"/>
+<via x="17.4625" y="17.4625" extent="1-16" drill="0.5" diameter="0.254"/>
 <contactref element="JP3" pad="1"/>
 <contactref element="C3" pad="2"/>
@@
 <via x="26.035" y="12.7" extent="1-16" drill="0.5" diameter="0.254"/>
 <via x="24.13" y="12.7" extent="1-16" drill="0.5" diameter="0.254"/>
+<wire x1="14.9225" y1="0.635" x2="13.0175" y2="7.3025" width="0" layer="19" extent="16-16"/>
 </signal>
 <signal name="AREF">
@@
 <signal name="SENSE_VCC">
 <contactref element="U2" pad="12"/>
-<contactref element="U$2" pad="VDD"/>
 <contactref element="R1" pad="1"/>
 <wire x1="25.4889" y1="7.5057" x2="25.4889" y2="3.1011" width="0.254" layer="16"/>
 <wire x1="25.4889" y1="3.1011" x2="26.05" y2="2.54" width="0.254" layer="16"/>
 <wire x1="26.05" y1="2.54" x2="26.05" y2="1.5725" width="0.254" layer="16"/>
-<wire x1="26.05" y1="1.5725" x2="26.67" y2="0.9525" width="0.254" layer="16"/>
 </signal>
 </signals>
