File: uV1/UKHASnet-avr-sensor.sch (EAGLE design)
At the start: 13 parts, among them J1 AVR_SPI_PRG_62X3_LOCK, U2 ATMEGA328P-AU

Commit message: Not much progress.
Parts:
- removed U$2: DS1820TO92, Ava:DS1820TO92
- added JP4: (no value), SparkFun-Connectors:M04PTH
Connections:
- net GND: no longer U$2.GND
- net SENSE1: no longer U$2.DQ
- net SENSE_VCC: no longer U$2.VCC
Changed lines of the file:
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@@
 <parts>
 <part name="U$1" library="hopeRF2" deviceset="RFM69HW" device=""/>
-<part name="U$2" library="Ava" deviceset="DS1820" device="TO92"/>
 <part name="J1" library="SparkFun-Connectors" deviceset="AVR_SPI_PRG_6" device="2X3_LOCK"/>
 <part name="U2" library="Ava" deviceset="ATMEGA328P-AU" device=""/>
@@
 <part name="JP1" library="SparkFun-Connectors" deviceset="M01" device="PTH"/>
 <part name="JP3" library="SparkFun-Connectors" deviceset="M01" device="PTH"/>
+<part name="JP4" library="SparkFun-Connectors" deviceset="M04" device="PTH"/>
 </parts>
 <sheets>
@@
 <instances>
 <instance part="U$1" gate="A" x="25.4" y="-22.86" rot="R180"/>
-<instance part="U$2" gate="G$1" x="-30.48" y="55.88" rot="R90"/>
 <instance part="J1" gate="G$1" x="104.14" y="104.14"/>
 <instance part="U2" gate="A" x="68.58" y="58.42"/>
@@
 <instance part="JP1" gate="G$1" x="-10.16" y="99.06"/>
 <instance part="JP3" gate="G$1" x="-10.16" y="83.82"/>
+<instance part="JP4" gate="G$1" x="-38.1" y="53.34"/>
 </instances>
 <busses>
@@
 </segment>
 <segment>
-<pinref part="U$2" gate="G$1" pin="DQ"/>
 <wire x1="-25.4" y1="55.88" x2="-20.32" y2="55.88" width="0.1524" layer="91"/>
 <label x="0" y="55.88" size="1.778" layer="95"/>
@@
 </segment>
 <segment>
-<pinref part="U$2" gate="G$1" pin="GND"/>
 <wire x1="-25.4" y1="53.34" x2="-20.32" y2="53.34" width="0.1524" layer="91"/>
 <label x="-10.16" y="53.34" size="1.778" layer="95"/>
@@
 </segment>
 <segment>
-<pinref part="U$2" gate="G$1" pin="VCC"/>
 <wire x1="-25.4" y1="58.42" x2="-22.86" y2="58.42" width="0.1524" layer="91"/>
 <wire x1="-22.86" y1="58.42" x2="-22.86" y2="66.04" width="0.1524" layer="91"/>
